Commit message: Evaluating on legos.

File: bullet/assets/lego.urdf (robot description, URDF)
Before this commit: robot cube.urdf, 1 links, 0 joints
Links:
- link legobrick: geometry collision box size=0.032 0.023 0.032; visual mesh filename=lego.obj scale=.5 .5 .5

Commit message: Get lego to be same size as boxes.

File: bullet/assets/lego.urdf (robot description, URDF)
Before this commit: robot cube.urdf, 1 links, 0 joints
Links:
- link legobrick: geometry collision box size=0.032 0.023 0.032; visual mesh filename=lego.obj scale=0.235 0.8 0.235

File: bullet/assets/lego_small.urdf (robot description, URDF)
Before this commit: robot cube.urdf, 1 links, 0 joints
Links:
- link legobrick: geometry collision box size=0.032 0.023 0.032; visual mesh filename=lego.obj scale=0.147 0.578 0.147

Commit message: Make lego (without studs) match the box height.

File: bullet/assets/lego.urdf (robot description, URDF)
Before this commit: robot cube.urdf, 1 links, 0 joints
Links:
- link legobrick: geometry collision box size=0.032 0.023 0.032; visual mesh filename=lego.obj scale=0.25 0.95 0.25

File: bullet/assets/lego_small.urdf (robot description, URDF)
Before this commit: robot cube.urdf, 1 links, 0 joints
Links:
- link legobrick: geometry collision box size=0.032 0.023 0.032; visual mesh filename=lego.obj scale=0.147 0.65 0.147
