Commit message: Working on debugging eval on irreg objects.

File: bullet/assets/cup/cup_small.urdf (robot description, URDF)
Before this commit: robot cube.urdf, 1 links, 0 joints
Links:
- link baseLink: geometry collision mesh filename=Cup/cup_vhacd.obj scale=0.5 0.5 0.5; visual mesh filename=Cup/textured-0008192.obj scale=1.5 1.5 1.5

Commit message: Get cup and lego dimensions to match large box.

File: bullet/assets/cup/cup_small.urdf (robot description, URDF)
Before this commit: robot cube.urdf, 1 links, 0 joints
Links:
- link baseLink: geometry collision mesh filename=Cup/cup_vhacd.obj scale=.5 .5 .5; visual mesh filename=Cup/textured-0008192.obj scale=.9 .9 1.3

File: bullet/assets/lego.urdf (robot description, URDF)
Before this commit: robot cube.urdf, 1 links, 0 joints
Links:
- link legobrick: geometry collision box size=0.032 0.023 0.032; visual mesh filename=lego.obj scale=.25 0.94 .25
